File: stm32f072c8tx_breakout.kicad_pcb (KiCad board)
At the start: 2 copper layers, 57.2 x 30 mm, 25 parts, among them J1 USB_OTG, J2 CONN_01X22, J3 CONN_01X22, J4 CONN_01X03, J5 CONN_01X04, SW1 SW_Push, U1 LM1117-3.3, U2 STM32F072C8Tx

Commit message: PCB changes
Parts:
- U1: footprint TO_SOT_Packages_SMD:SOT-223 -> TO_SOT_Packages_SMD:SOT-223-3Lead_TabPin2
- moved C2 1.82 mm to (135.2, 113.2)
- moved C4 0.79 mm to (124.8, 121.8), turned to 315 degrees
- moved C8 0.56 mm to (133.8, 116.8), turned to 45 degrees
- moved C6 0.35 mm to (131.2, 108.2)
Connections:
- J3 pad 10: /PB3 -> /PA15
- J3 pad 11: /PA15 -> /PA12
- J3 pad 12: /PA12 -> /PA11
- J3 pad 13: /PA11 -> /PA10
- J3 pad 14: /PA10 -> /PA9
- J3 pad 15: /PA9 -> /PA8
- J3 pad 16: /PA8 -> /PB15
- J3 pad 17: /PB15 -> /PB14
- J3 pad 18: /PB14 -> /PB13
- J3 pad 19: /PB13 -> /PB12
- J3 pad 20: /PB12 -> VDD
- J3 pad 21: VDD -> GND
- J3 pad 22: GND -> +5V
- J3 pad 3: +5V -> /PB9
- J3 pad 4: /PB9 -> /PB8
- J3 pad 5: /PB8 -> /PB7
- J3 pad 6: /PB7 -> /PB6
- J3 pad 7: /PB6 -> /PB5
- J3 pad 8: /PB5 -> /PB4
- J3 pad 9: /PB4 -> /PB3
Routing:
- net GND: track 197.4 -> 228.0 mm, vias 7 -> 9
- net +5V: track 55.1 -> 33.8 mm
- net /SYS_SWCLK: track 32.3 -> 37.4 mm
- net /PA12: track 37.6 -> 41.1 mm
- net /PB14: track 19.2 -> 15.7 mm
- net /PB13: track 21.3 -> 18.1 mm
- net /PB12: track 23.6 -> 20.4 mm
- net /PA11: track 34.8 -> 37.8 mm
- net /SYS_SWDIO: track 32.3 -> 34.8 mm
- net /PB6: track 13.7 -> 16.1 mm
- net /PB7: track 16.2 -> 18.5 mm
- net /PB15: track 16.7 -> 14.5 mm
- net /PB8: track 18.6 -> 20.6 mm
- net /PB9: track 21.2 -> 22.9 mm
- net /PB5: track 12.4 -> 13.8 mm
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Other:
- board text added: "RESET"
- board text removed: "Reset"
