File: stm32f072c8tx_breakout.sch (KiCad schematic (older format))
At the start: 25 parts, among them J1 USB_OTG, J2 CONN_01X22, J3 CONN_01X22, J4 CONN_01X03, J5 CONN_01X04, SW1 SW_Push, U1 LM1117-3.3, U2 STM32F072C8Tx

Commit message: PCB changes
Parts:
- U1: footprint TO_SOT_Packages_SMD:SOT-223 -> TO_SOT_Packages_SMD:SOT-223-3Lead_TabPin2
Changed lines of the file:
@@
 Text Label 14900 2050 0    60   ~ 0
 GND
+Text Label 14900 4050 0    60   ~ 0
++5V
 Text Label 14900 2150 0    60   ~ 0
-+5V
+PB9
 Text Label 14900 2250 0    60   ~ 0
-PB9
+PB8
 Text Label 14900 2350 0    60   ~ 0
-PB8
+PB7
 Text Label 14900 2450 0    60   ~ 0
-PB7
+PB6
 Text Label 14900 2550 0    60   ~ 0
-PB6
+PB5
 Text Label 14900 2650 0    60   ~ 0
-PB5
+PB4
 Text Label 14900 2750 0    60   ~ 0
-PB4
+PB3
 Text Label 14900 2850 0    60   ~ 0
-PB3
+PA15
 Text Label 14900 2950 0    60   ~ 0
-PA15
+PA12
 Text Label 14900 3050 0    60   ~ 0
-PA12
+PA11
 Text Label 14900 3150 0    60   ~ 0
-PA11
+PA10
 Text Label 14900 3250 0    60   ~ 0
-PA10
+PA9
 Text Label 14900 3350 0    60   ~ 0
-PA9
+PA8
 Text Label 14900 3450 0    60   ~ 0
-PA8
+PB15
 Text Label 14900 3550 0    60   ~ 0
-PB15
+PB14
 Text Label 14900 3650 0    60   ~ 0
-PB14
+PB13
 Text Label 14900 3750 0    60   ~ 0
-PB13
-Text Label 14900 3850 0    60   ~ 0
 PB12
 Text Label 13250 8300 0    60   ~ 0
@@
 F 0 "U1" H 2450 7767 50  0000 C CNN
 F 1 "LM1117-3.3" H 2450 7676 50  0000 C CNN
-F 2 "TO_SOT_Packages_SMD:SOT-223" H 2450 7400 50  0001 C CNN
+F 2 "TO_SOT_Packages_SMD:SOT-223-3Lead_TabPin2" H 2450 7400 50  0001 C CNN
 F 3 "" H 2450 7400 50  0001 C CNN
 	1    2450 7400
@@
 	15450 2050 14750 2050
 Wire Wire Line
+	15450 4050 14750 4050
+Wire Wire Line
 	15450 2150 14750 2150
 Wire Wire Line
@@
 Wire Wire Line
 	15450 3750 14750 3750
-Wire Wire Line
-	15450 3850 14750 3850
 Wire Wire Line
 	13800 8300 13100 8300
@@
 	-1   0    0    -1
 $EndComp
+Text Label 14900 3850 0    60   ~ 0
+VDD
 Text Label 14900 3950 0    60   ~ 0
-VDD
-Text Label 14900 4050 0    60   ~ 0
 GND
 Wire Wire Line
+	15450 3850 14750 3850
+Wire Wire Line
 	15450 3950 14750 3950
-Wire Wire Line
-	15450 4050 14750 4050
 $EndSCHEMATC
